File: BrickBase/hardware/BrickBase.kicad_sch (KiCad schematic)
At the start: 11 parts, among them J1 RJ12, J2 RJ12, J3 RJ12, J4 RJ12, J5 RJ12, J6 RJ12, J7 Conn_01x19, J8 Conn_01x19, U1 PCA9306D

Commit message: .
Other:
- note added: "29-apr-2025"
- note added: "BrickBase"
Changed lines of the file:
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@@
+		)
+	)
+	(text "BrickBase"
+		(exclude_from_sim no)
+		(at 194.564 173.736 0)
+		(effects
+			(font
+				(size 3.81 3.81)
+			)
+		)
+	)
+	(text "29-apr-2025"
+		(exclude_from_sim no)
+		(at 213.614 193.294 0)
+		(effects
+			(font
+				(size 1.27 1.27)
+			)
 		)
 	)
